Commit message: Remove base_joint from macro for flexibility

File: robotiq_2f_85_description/urdf/robotiq_2f_85.urdf.xacro (robot description, xacro)
@@ -5,7 +5,10 @@
     <!-- Import macro -->
     <xacro:include filename="$(find robotiq_2f_85_description)/urdf/robotiq_2f_85_macro.xacro" />
+    <xacro:robotiq_2f_85 prefix="$(arg prefix)" />
     <link name="world" />
-    <xacro:robotiq_2f_85 parent="world" prefix="$(arg prefix)">
+    <joint name="$(arg prefix)base_joint" type="fixed">
+        <parent link="world" />
+        <child link="$(arg prefix)base_link" />
         <origin xyz="0 0 0" rpy="0 0 0" />
-    </xacro:robotiq_2f_85>
+    </joint>
 </robot>

File: robotiq_2f_85_description/urdf/robotiq_2f_85_macro.xacro (robot description, xacro)
@@ -1,5 +1,5 @@
 <?xml version="1.0"?>
 <robot xmlns:xacro="http://wiki.ros.org/xacro">
-    <xacro:macro name="robotiq_2f_85" params="parent *origin prefix">
+    <xacro:macro name="robotiq_2f_85" params="prefix">
         <xacro:property name="description_package" value="file://$(find robotiq_2f_85_description)" />
         <link name="${prefix}base_link">
@@ -20,9 +20,4 @@
             </inertial>
         </link>
-        <joint name="${prefix}base_joint" type="fixed">
-            <parent link="${parent}" />
-            <child link="${prefix}base_link" />
-            <xacro:insert_block name="origin" />
-        </joint>
         <!-- Macro to define a single finger -->
         <xacro:macro name="finger" params="finger mirror">

Commit message: Add UR coupling option

File: robotiq_2f_85_description/urdf/robotiq_2f_85.urdf.xacro (robot description, xacro)
@@ -1,14 +1,22 @@
 <?xml version="1.0"?>
 <robot xmlns:xacro="http://wiki.ros.org/xacro" name="robotiq_2f_85">
-    <!-- parameters -->
+    <!-- Parameters -->
     <xacro:arg name="prefix" default="robotiq_2f_" />
+    <xacro:arg name="ur_coupling" default="false" />
     <!-- Import macro -->
     <xacro:include filename="$(find robotiq_2f_85_description)/urdf/robotiq_2f_85_macro.xacro" />
-    <xacro:robotiq_2f_85 prefix="$(arg prefix)" />
+    <xacro:robotiq_2f_85 prefix="$(arg prefix)" ur_coupling="$(arg ur_coupling)" />
+    <!-- Joint with world -->
     <link name="world" />
-    <joint name="$(arg prefix)base_joint" type="fixed">
+    <xacro:if value="$(arg ur_coupling)">
+        <xacro:property name="root_link" value="$(arg prefix)coupling_link" />
+    </xacro:if>
+    <xacro:unless value="$(arg ur_coupling)">
+        <xacro:property name="root_link" value="$(arg prefix)base_link" />
+    </xacro:unless>
+    <joint name="$(arg prefix)root_joint" type="fixed">
         <parent link="world" />
-        <child link="$(arg prefix)base_link" />
-        <origin xyz="0 0 0" rpy="0 0 0" />
+        <child link="${root_link}" />
+        <origin xyz="0 0 0.01" rpy="0 0 0" />
     </joint>
 </robot>

File: robotiq_2f_85_description/urdf/robotiq_2f_85_macro.xacro (robot description, xacro)
@@ -1,5 +1,5 @@
 <?xml version="1.0"?>
 <robot xmlns:xacro="http://wiki.ros.org/xacro">
-    <xacro:macro name="robotiq_2f_85" params="prefix">
+    <xacro:macro name="robotiq_2f_85" params="prefix ur_coupling:=false">
         <xacro:property name="description_package" value="file://$(find robotiq_2f_85_description)" />
         <link name="${prefix}base_link">
@@ -20,4 +20,28 @@
             </inertial>
         </link>
+        <xacro:if value="${ur_coupling}">
+            <link name="${prefix}coupling_link">
+                <visual>
+                    <geometry>
+                        <mesh filename="${description_package}/meshes/visual/grp_es_cpl_062.dae" />
+                    </geometry>
+                </visual>
+                <collision>
+                    <geometry>
+                        <mesh filename="${description_package}/meshes/collision/grp_es_cpl_062.stl" />
+                    </geometry>
+                </collision>
+                <inertial>
+                    <origin xyz="-0.9e-3 0.0 5.26e-3" rpy="0 0 0" />
+                    <mass value="0.100" />
+                    <inertia ixx="40.8e-6" iyy="42.9e-6" izz="80.7e-6" ixy="0.4e-6" ixz="-0.1e-6" iyz="0.2e-6" />
+                </inertial>
+            </link>
+            <joint name="${prefix}base_joint" type="fixed">
+                <parent link="${prefix}coupling_link" />
+                <child link="${prefix}base_link" />
+                <origin xyz="0 0 11e-3" rpy="0 0 0" />
+            </joint>
+        </xacro:if>
         <!-- Macro to define a single finger -->
         <xacro:macro name="finger" params="finger mirror">

Commit message: Include ros2_control macro
Add property "name"
Put "file://" out of property "description_package"

File: robotiq_2f_85_description/urdf/robotiq_2f_85.urdf.xacro (robot description, xacro)
@@ -6,5 +6,5 @@
     <!-- Import macro -->
     <xacro:include filename="$(find robotiq_2f_85_description)/urdf/robotiq_2f_85_macro.xacro" />
-    <xacro:robotiq_2f_85 prefix="$(arg prefix)" ur_coupling="$(arg ur_coupling)" />
+    <xacro:robotiq_2f_85 name="robotiq_2f_85" prefix="$(arg prefix)" ur_coupling="$(arg ur_coupling)" />
     <!-- Joint with world -->
     <link name="world" />

File: robotiq_2f_85_description/urdf/robotiq_2f_85_macro.xacro (robot description, xacro)
@@ -1,15 +1,18 @@
 <?xml version="1.0"?>
 <robot xmlns:xacro="http://wiki.ros.org/xacro">
-    <xacro:macro name="robotiq_2f_85" params="prefix ur_coupling:=false">
-        <xacro:property name="description_package" value="file://$(find robotiq_2f_85_description)" />
+    <xacro:macro name="robotiq_2f_85" params="name prefix ur_coupling:=false">
+        <xacro:property name="description_package" value="$(find robotiq_2f_85_description)" />
+        <!-- ros2_control -->
+        <xacro:include filename="${description_package}/urdf/robotiq_2f_85.ros2_control.xacro" />
+        <xacro:robotiq_2f_85_ros2_control name="${name}" prefix="${prefix}" />
         <link name="${prefix}base_link">
             <visual>
                 <geometry>
-                    <mesh filename="${description_package}/meshes/visual/base.dae" />
+                    <mesh filename="file://${description_package}/meshes/visual/base.dae" />
                 </geometry>
             </visual>
             <collision>
                 <geometry>
-                    <mesh filename="${description_package}/meshes/collision/base.stl" />
+                    <mesh filename="file://${description_package}/meshes/collision/base.stl" />
                 </geometry>
             </collision>
@@ -24,10 +27,10 @@
                 <visual>
                     <geometry>
-                        <mesh filename="${description_package}/meshes/visual/grp_es_cpl_062.dae" />
+                        <mesh filename="file://${description_package}/meshes/visual/grp_es_cpl_062.dae" />
                     </geometry>
                 </visual>
                 <collision>
                     <geometry>
-                        <mesh filename="${description_package}/meshes/collision/grp_es_cpl_062.stl" />
+                        <mesh filename="file://${description_package}/meshes/collision/grp_es_cpl_062.stl" />
                     </geometry>
                 </collision>
@@ -57,10 +60,10 @@
                 <visual>
                     <geometry>
-                        <mesh filename="${description_package}/meshes/visual/fingertip.dae" />
+                        <mesh filename="file://${description_package}/meshes/visual/fingertip.dae" />
                     </geometry>
                 </visual>
                 <collision>
                     <geometry>
-                        <mesh filename="${description_package}/meshes/collision/fingertip.stl" />
+                        <mesh filename="file://${description_package}/meshes/collision/fingertip.stl" />
                     </geometry>
                 </collision>
@@ -74,10 +77,10 @@
                 <visual>
                     <geometry>
-                        <mesh filename="${description_package}/meshes/visual/finger1.dae" />
+                        <mesh filename="file://${description_package}/meshes/visual/finger1.dae" />
                     </geometry>
                 </visual>
                 <collision>
                     <geometry>
-                        <mesh filename="${description_package}/meshes/collision/finger1.stl" />
+                        <mesh filename="file://${description_package}/meshes/collision/finger1.stl" />
                     </geometry>
                 </collision>
@@ -91,10 +94,10 @@
                 <visual>
                     <geometry>
-                        <mesh filename="${description_package}/meshes/visual/finger2.dae" />
+                        <mesh filename="file://${description_package}/meshes/visual/finger2.dae" />
                     </geometry>
                 </visual>
                 <collision>
                     <geometry>
-                        <mesh filename="${description_package}/meshes/collision/finger2.stl" />
+                        <mesh filename="file://${description_package}/meshes/collision/finger2.stl" />
                     </geometry>
                 </collision>
@@ -108,10 +111,10 @@
                 <visual>
                     <geometry>
-                        <mesh filename="${description_package}/meshes/visual/finger3.dae" />
+                        <mesh filename="file://${description_package}/meshes/visual/finger3.dae" />
                     </geometry>
                 </visual>
                 <collision>
                     <geometry>
-                        <mesh filename="${description_package}/meshes/collision/finger3.stl" />
+                        <mesh filename="file://${description_package}/meshes/collision/finger3.stl" />
                     </geometry>
                 </collision>
@@ -125,10 +128,10 @@
                 <visual>
                     <geometry>
-                        <mesh filename="${description_package}/meshes/visual/finger4.dae" />
+                        <mesh filename="file://${description_package}/meshes/visual/finger4.dae" />
                     </geometry>
                 </visual>
                 <collision>
                     <geometry>
-                        <mesh filename="${description_package}/meshes/collision/finger4.stl" />
+                        <mesh filename="file://${description_package}/meshes/collision/finger4.stl" />
                     </geometry>
                 </collision>

Commit message: Add mimic joints option

File: robotiq_2f_85_description/urdf/robotiq_2f_85.urdf.xacro (robot description, xacro)
@@ -4,7 +4,13 @@
     <xacro:arg name="prefix" default="robotiq_2f_" />
     <xacro:arg name="ur_coupling" default="false" />
+    <xacro:arg name="mimic" default="true" />
     <!-- Import macro -->
     <xacro:include filename="$(find robotiq_2f_85_description)/urdf/robotiq_2f_85_macro.xacro" />
-    <xacro:robotiq_2f_85 name="robotiq_2f_85" prefix="$(arg prefix)" ur_coupling="$(arg ur_coupling)" />
+    <xacro:robotiq_2f_85
+        name="robotiq_2f_85"
+        prefix="$(arg prefix)"
+        ur_coupling="$(arg ur_coupling)"
+        mimic="$(arg mimic)"
+    />
     <!-- Joint with world -->
     <link name="world" />

File: robotiq_2f_85_description/urdf/robotiq_2f_85_macro.xacro (robot description, xacro)
@@ -1,5 +1,5 @@
 <?xml version="1.0"?>
 <robot xmlns:xacro="http://wiki.ros.org/xacro">
-    <xacro:macro name="robotiq_2f_85" params="name prefix ur_coupling:=false">
+    <xacro:macro name="robotiq_2f_85" params="name prefix ur_coupling:=false mimic:=true">
         <xacro:property name="description_package" value="$(find robotiq_2f_85_description)" />
         <!-- ros2_control -->
@@ -153,4 +153,7 @@
                 <origin xyz="${x_gain * 30.60114e-3} 0.0 54.90452e-3" rpy="0 0 ${yaw}" />
                 <limit lower="0.0" upper="0.8" velocity="0.5" effort="50" />
+                <xacro:if value="${mimic and mirror}">
+                    <mimic joint="${prefix}left_finger1_joint" />
+                </xacro:if>
             </joint>
             <joint name="${prefix}${finger}_finger2_joint" type="fixed">
@@ -164,4 +167,7 @@
                 <axis xyz="0 -1 0" />
                 <origin xyz="${x_gain * 12.7e-3} 0.0 61.42e-3" rpy="0 0 ${yaw}" />
+                <xacro:if value="${mimic}">
+                    <mimic joint="${prefix}${finger}_finger1_joint" />
+                </xacro:if>
             </joint>
             <joint name="${prefix}${finger}_finger4-2_joint" type="continuous">
@@ -170,16 +176,21 @@
                 <axis xyz="0 -1 0" />
                 <origin xyz="4.30896e-3 0.0 47.39022e-3" rpy="0 0 0" />
+                <xacro:if value="${mimic}">
+                    <mimic joint="${prefix}${finger}_finger1_joint" multiplier="-1" />
+                </xacro:if>
             </joint>
-            <!-- Close loop by injecting SDF -->
-            <gazebo>
-                <joint name="${prefix}${finger}_finger4-3_joint" type="revolute">
-                    <parent>${prefix}${finger}_finger3_link</parent>
-                    <child>${prefix}${finger}_finger4_link</child>
-                    <axis>
-                        <xyz>0 -1 0</xyz>
-                    </axis>
-                    <pose>-17.90144e-3 0.0 6.51468e-3 0 0 0</pose>
-                </joint>
-            </gazebo>
+            <xacro:unless value="${mimic}">
+                <!-- Close loop by injecting SDF -->
+                <gazebo>
+                    <joint name="${prefix}${finger}_finger4-3_joint" type="revolute">
+                        <parent>${prefix}${finger}_finger3_link</parent>
+                        <child>${prefix}${finger}_finger4_link</child>
+                        <axis>
+                            <xyz>0 -1 0</xyz>
+                        </axis>
+                        <pose>-17.90144e-3 0.0 6.51468e-3 0 0 0</pose>
+                    </joint>
+                </gazebo>
+            </xacro:unless>
         </xacro:macro>
         <xacro:finger finger="left" mirror="false" />
