Commit message: Add mock interface for ros2_control
- Cleanup interface definitions

File: robotiq_2f_85_description/urdf/robotiq_2f_85.ros2_control.xacro (robot description, xacro)
@@ -1,23 +1,20 @@
 <?xml version="1.0"?>
 <robot xmlns:xacro="http://wiki.ros.org/xacro">
-    <xacro:macro name="robotiq_2f_85_ros2_control" params="name prefix">
+    <xacro:macro name="robotiq_2f_85_ros2_control" params="name prefix sim_gazebo">
         <ros2_control name="${name}" type="system">
             <hardware>
-                <plugin>gazebo_ros2_control/GazeboSystem</plugin>
+                <xacro:unless value="${sim_gazebo}">
+                    <plugin>mock_components/GenericSystem</plugin>
+                </xacro:unless>
+                <xacro:if value="${sim_gazebo}">
+                    <plugin>gazebo_ros2_control/GazeboSystem</plugin>
+                </xacro:if>
             </hardware>
             <xacro:macro name="finger_ros2_control" params="finger">
                 <joint name="${prefix}${finger}_finger1_joint">
-                    <command_interface name="effort" />
-                    <state_interface name="position" />
-                    <state_interface name="velocity" />
-                    <state_interface name="effort" />
-                </joint>
-                <joint name="${prefix}${finger}_finger3_joint">
-                    <state_interface name="position" />
-                    <state_interface name="velocity" />
-                </joint>
-                <joint name="${prefix}${finger}_finger4-2_joint">
-                    <state_interface name="position" />
-                    <state_interface name="velocity" />
+                    <command_interface name="position" />
+                    <state_interface name="position">
+                        <param name="initial_value">0.0</param>
+                    </state_interface>
                 </joint>
             </xacro:macro>

File: robotiq_2f_85_description/urdf/robotiq_2f_85.urdf.xacro (robot description, xacro)
@@ -5,4 +5,5 @@
     <xacro:arg name="ur_coupling" default="false" />
     <xacro:arg name="mimic" default="true" />
+    <xacro:arg name="sim_gazebo" default="false" />
     <!-- Import macro -->
     <xacro:include filename="$(find robotiq_2f_85_description)/urdf/robotiq_2f_85_macro.xacro" />
@@ -12,4 +13,5 @@
         ur_coupling="$(arg ur_coupling)"
         mimic="$(arg mimic)"
+        sim_gazebo="$(arg sim_gazebo)"
     />
     <!-- Joint with world -->

File: robotiq_2f_85_description/urdf/robotiq_2f_85_macro.xacro (robot description, xacro)
@@ -1,9 +1,9 @@
 <?xml version="1.0"?>
 <robot xmlns:xacro="http://wiki.ros.org/xacro">
-    <xacro:macro name="robotiq_2f_85" params="name prefix ur_coupling:=false mimic:=true">
+    <xacro:macro name="robotiq_2f_85" params="name prefix ur_coupling:=false mimic:=true sim_gazebo:=false">
         <xacro:property name="description_package" value="$(find robotiq_2f_85_description)" />
         <!-- ros2_control -->
         <xacro:include filename="${description_package}/urdf/robotiq_2f_85.ros2_control.xacro" />
-        <xacro:robotiq_2f_85_ros2_control name="${name}" prefix="${prefix}" />
+        <xacro:robotiq_2f_85_ros2_control name="${name}" prefix="${prefix}" sim_gazebo="${sim_gazebo}" />
         <link name="${prefix}base_link">
             <visual>
